File: Hydra/Hydra.kicad_sch (KiCad schematic)
At the start: 116 parts, among them J1 USB_C_Receptacle_USB2.0, SW1 SW_Push, U1 USBLC6-2SC6, U2 ATmega32U4-M, Y1 16MHz

Commit message: Fixed Matrix
Connections:
- net ROW1: no longer D28.1 (K)
- net ROW2: now also D28.1 (K), D31.1 (K), D35.1 (K), D39.1 (K), D43.1 (K)
- net ROW3: now also D32.1 (K), D36.1 (K), D40.1 (K), D44.1 (K)
Changed lines of the file:
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@@
   (junction (at 119.38 45.085) (diameter 0) (color 0 0 0 0)
   )
+  (junction (at 109.22 76.2) (diameter 0) (color 0 0 0 0)
+  )
   (junction (at 144.145 137.16) (diameter 0) (color 0 0 0 0)
   )
@@
   (junction (at 63.5 76.2) (diameter 0) (color 0 0 0 0)
   )
+  (junction (at 109.22 64.135) (diameter 0) (color 0 0 0 0)
+  )
   (junction (at 117.475 52.07) (diameter 0) (color 0 0 0 0)
   )
@@
   (junction (at 236.855 19.05) (diameter 0) (color 0 0 0 0)
   )
+  (junction (at 80.01 77.47) (diameter 0) (color 0 0 0 0)
+  )
   (junction (at 127.635 57.15) (diameter 0) (color 0 0 0 0)
   )
@@
   (junction (at 182.245 43.18) (diameter 0) (color 0 0 0 0)
   )
+  (junction (at 100.33 64.135) (diameter 0) (color 0 0 0 0)
+  )
   (junction (at 126.365 52.07) (diameter 0) (color 0 0 0 0)
   )
   (junction (at 63.5 52.07) (diameter 0) (color 0 0 0 0)
   )
-  (junction (at 90.805 64.135) (diameter 0) (color 0 0 0 0)
+  (junction (at 81.28 66.04) (diameter 0) (color 0 0 0 0)
   )
   (junction (at 55.245 64.135) (diameter 0) (color 0 0 0 0)
@@
     (stroke (width 0) (type default) (color 0 0 0 0))
   )
+  (wire (pts (xy 80.01 77.47) (xy 80.01 76.2))
+    (stroke (width 0) (type default) (color 0 0 0 0))
+  )
   (wire (pts (xy 91.44 69.215) (xy 91.44 81.28))
     (stroke (width 0) (type default) (color 0 0 0 0))
@@
     (stroke (width 0) (type default) (color 0 0 0 0))
   )
+  (wire (pts (xy 100.33 66.04) (xy 81.28 66.04))
+    (stroke (width 0) (type default) (color 0 0 0 0))
+  )
   (wire (pts (xy 81.28 88.265) (xy 80.01 88.265))
     (stroke (width 0) (type default) (color 0 0 0 0))
@@
     (stroke (width 0) (type default) (color 0 0 0 0))
   )
+  (wire (pts (xy 106.045 76.2) (xy 106.045 77.47))
+    (stroke (width 0) (type default) (color 0 0 0 0))
+  )
   (wire (pts (xy 144.145 134.62) (xy 144.145 137.16))
     (stroke (width 0) (type default) (color 0 0 0 0))
@@
     (stroke (width 0) (type default) (color 0 0 0 0))
   )
+  (wire (pts (xy 100.33 64.135) (xy 100.33 66.04))
+    (stroke (width 0) (type default) (color 0 0 0 0))
+  )
   (wire (pts (xy 37.465 74.295) (xy 37.465 76.2))
     (stroke (width 0) (type default) (color 0 0 0 0))
@@
     (stroke (width 0) (type default) (color 0 0 0 0))
   )
+  (wire (pts (xy 100.33 64.135) (xy 109.22 64.135))
+    (stroke (width 0) (type default) (color 0 0 0 0))
+  )
   (wire (pts (xy 82.55 22.86) (xy 82.55 33.02))
     (stroke (width 0) (type default) (color 0 0 0 0))
@@
     (stroke (width 0) (type default) (color 0 0 0 0))
   )
+  (wire (pts (xy 109.22 76.2) (xy 106.045 76.2))
+    (stroke (width 0) (type default) (color 0 0 0 0))
+  )
   (wire (pts (xy 81.28 52.07) (xy 100.33 52.07))
     (stroke (width 0) (type default) (color 0 0 0 0))
@@
     (stroke (width 0) (type default) (color 0 0 0 0))
   )
-  (wire (pts (xy 80.01 88.265) (xy 80.01 76.2))
+  (wire (pts (xy 80.01 88.265) (xy 80.01 77.47))
     (stroke (width 0) (type default) (color 0 0 0 0))
   )
@@
     (stroke (width 0) (type default) (color 0 0 0 0))
   )
-  (wire (pts (xy 90.805 64.135) (xy 100.33 64.135))
-    (stroke (width 0) (type default) (color 0 0 0 0))
-  )
   (wire (pts (xy 203.2 31.115) (xy 205.74 31.115))
     (stroke (width 0) (type default) (color 0 0 0 0))
@@
     (stroke (width 0) (type default) (color 0 0 0 0))
   )
+  (wire (pts (xy 106.045 77.47) (xy 80.01 77.47))
+    (stroke (width 0) (type default) (color 0 0 0 0))
+  )

Commit message: mcu traces
Connections:
- net at R4.2: now also U2.3 (D-); no longer U2.4 (D+)
- net at R5.2: now also U2.4 (D+); no longer U2.3 (D-)
Other:
- moved on the sheet: R4, R5
Changed lines of the file:
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@@
     )
   )
-  (global_label "D+" (shape input) (at 194.31 59.055 180) (fields_autoplaced)
+  (global_label "D+" (shape input) (at 194.31 56.515 180) (fields_autoplaced)
     (effects (font (size 1.27 1.27)) (justify right))
-    (property "Intersheet References" "${INTERSHEET_REFS}" (id 0) (at 189.0545 59.1344 0)
+    (property "Intersheet References" "${INTERSHEET_REFS}" (id 0) (at 189.0545 56.5944 0)
       (effects (font (size 1.27 1.27)) (justify right) hide)
     )
@@
     )
   )
-  (global_label "D-" (shape input) (at 194.31 56.515 180) (fields_autoplaced)
+  (global_label "D-" (shape input) (at 194.31 59.055 180) (fields_autoplaced)
     (effects (font (size 1.27 1.27)) (justify right))
-    (property "Intersheet References" "${INTERSHEET_REFS}" (id 0) (at 189.0545 56.4356 0)
+    (property "Intersheet References" "${INTERSHEET_REFS}" (id 0) (at 189.0545 58.9756 0)
       (effects (font (size 1.27 1.27)) (justify right) hide)
     )
@@
     (pin "2")
   )
-  (symbol (lib_id "Device:R_Small") (at 207.645 56.515 90) (unit 1)
-    (in_bom yes) (on_board yes) (fields_autoplaced)
-    (property "Reference" "R4" (id 0) (at 207.645 50.8 90))
-    (property "Value" "22" (id 1) (at 207.645 53.34 90))
-    (property "Footprint" "Resistor_SMD:R_0805_2012Metric" (id 2) (at 207.645 56.515 0)
-      (effects (font (size 1.27 1.27)) hide)
-    )
-    (property "Datasheet" "~" (id 3) (at 207.645 56.515 0)
+  (symbol (lib_id "Device:R_Small") (at 207.645 59.055 90) (unit 1)
+    (in_bom yes) (on_board yes) (fields_autoplaced)
+    (property "Reference" "R4" (id 0) (at 207.645 53.34 90))
+    (property "Value" "22" (id 1) (at 207.645 55.88 90))
+    (property "Footprint" "Resistor_SMD:R_0805_2012Metric" (id 2) (at 207.645 59.055 0)
+      (effects (font (size 1.27 1.27)) hide)
+    )
+    (property "Datasheet" "~" (id 3) (at 207.645 59.055 0)
       (effects (font (size 1.27 1.27)) hide)
     )
@@
     (pin "2")
   )
-  (symbol (lib_id "Device:R_Small") (at 207.645 59.055 90) (unit 1)
+  (symbol (lib_id "Device:R_Small") (at 207.645 56.515 90) (unit 1)
     (in_bom yes) (on_board yes)
-    (property "Reference" "R5" (id 0) (at 207.645 62.23 90))
-    (property "Value" "22" (id 1) (at 207.645 64.77 90))
-    (property "Footprint" "Resistor_SMD:R_0805_2012Metric" (id 2) (at 207.645 59.055 0)
-      (effects (font (size 1.27 1.27)) hide)
-    )
-    (property "Datasheet" "~" (id 3) (at 207.645 59.055 0)
-      (effects (font (size 1.27 1.27)) hide)
-    )
+    (property "Reference" "R5" (id 0) (at 207.645 59.69 90))
+    (property "Value" "22" (id 1) (at 207.645 62.23 90))
+    (property "Footprint" "Resistor_SMD:R_0805_2012Metric" (id 2) (at 207.645 56.515 0)
+      (effects (font (size 1.27 1.27)) hide)
+    )
+    (property "Datasheet" "~" (id 3) (at 207.645 56.515 0)
+      (effects (font (size 1.27 1.27)) hide)
+    )
