File: Hydra/Hydra.kicad_sch (KiCad schematic)
At the start: 117 parts, among them J1 USB_C_Receptacle_USB2.0, SW1 SW_Push, U1 USBLC6-2SC6, U2 ATmega32U4-M, Y1 16MHz

Commit message: finished mcu routes
Parts:
- Brd1: renamed from Brd?; footprint (none) -> SSD1306:128x64OLED
Changed lines of the file:
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@@
   (symbol (lib_id "SSD1306-128x64_OLED:SSD1306") (at 162.56 100.33 0) (unit 1)
     (in_bom yes) (on_board yes) (fields_autoplaced)
-    (property "Reference" "Brd?" (id 0) (at 170.18 99.0599 0)
+    (property "Reference" "Brd1" (id 0) (at 170.18 99.0599 0)
       (effects (font (size 1.27 1.27)) (justify left))
     )
@@
       (effects (font (size 1.27 1.27)) (justify left))
     )
-    (property "Footprint" "" (id 2) (at 162.56 93.98 0)
+    (property "Footprint" "SSD1306:128x64OLED" (id 2) (at 162.56 93.98 0)
       (effects (font (size 1.27 1.27)) hide)
     )
@@
   (symbol (lib_id "power:+5V") (at 161.29 87.63 0) (unit 1)
     (in_bom yes) (on_board yes) (fields_autoplaced)
-    (property "Reference" "#PWR?" (id 0) (at 161.29 91.44 0)
+    (property "Reference" "#PWR0116" (id 0) (at 161.29 91.44 0)
       (effects (font (size 1.27 1.27)) hide)
     )
@@
   (symbol (lib_id "power:GND") (at 152.4 91.44 0) (unit 1)
     (in_bom yes) (on_board yes) (fields_autoplaced)
-    (property "Reference" "#PWR?" (id 0) (at 152.4 97.79 0)
+    (property "Reference" "#PWR0117" (id 0) (at 152.4 97.79 0)
       (effects (font (size 1.27 1.27)) hide)
     )
@@
     )
     (path "/890da6e5-452a-4cee-97d4-bc293bca2484"
-      (reference "#PWR?") (unit 1) (value "+5V") (footprint "")
+      (reference "#PWR0116") (unit 1) (value "+5V") (footprint "")
     )
     (path "/bb077c81-5259-4a82-acd6-a0cbee4fd534"
-      (reference "#PWR?") (unit 1) (value "GND") (footprint "")
+      (reference "#PWR0117") (unit 1) (value "GND") (footprint "")
     )
     (path "/0acc27a1-140c-44c7-bc97-805be210a998"
-      (reference "Brd?") (unit 1) (value "SSD1306") (footprint "")
+      (reference "Brd1") (unit 1) (value "SSD1306") (footprint "SSD1306:128x64OLED")
     )
     (path "/c2c25ddc-a213-459b-81d0-110e8fa44967"

Commit message: Added 2 1u options for space
Parts:
- added D45, D46, D47, D48: D_Small, Diode_SMD:D_SOD-123, symbol Device:D_Small
- added MX45, MX46, MX47, MX48: MX-NoLED, MX_Only:MXOnly-1U-NoLED, symbol MX_Alps_Hybrid:MX-NoLED
Connections:
- net COL4: now also MX45.1 (COL)
- net COL5: now also MX46.1 (COL)
- net COL6: now also MX47.1 (COL)
- net COL7: now also MX48.1 (COL)
- net ROW0: now also D20.1 (K), D23.1 (K)
- net ROW1: now also D21.1 (K), D24.1 (K); no longer D20.1 (K), D23.1 (K)
- net ROW2: now also D22.1 (K), D25.1 (K); no longer D21.1 (K), D24.1 (K)
- net ROW3: now also D45.1 (K), D46.1 (K), D47.1 (K), D48.1 (K); no longer D22.1 (K), D25.1 (K)
- new net: D47.2 (A), MX47.2 (ROW)
- new net: D46.2 (A), MX46.2 (ROW)
- new net: D45.2 (A), MX45.2 (ROW)
- new net: D48.2 (A), MX48.2 (ROW)
