File: Hydra/Hydra.kicad_pcb (KiCad board)
At the start: 2 copper layers, 116 parts, among them J1 USB_C_Receptacle_USB2.0, SW1 SW_Push, U1 USBLC6-2SC6, U2 ATmega32U4-M, Y1 16MHz

Commit message: finished layout placed diodes
Parts:
- D1, D10, D11, D12, D13, D14, D15, D16, D17, D18, D19, D2, D20, D21, D22, D23, D24, D26, D27, D28, D29, D3, D30, D31, D32, D33, D34, D35, D36, D37, D38, D39, D4, D40, D41, D42, D43, D44, D5, D6, D7, D8, D9: moved to B.Cu
- moved D41 316.8 mm to (283.0, 66.5), turned to 180 degrees
- moved MX39 299.3 mm to (257.2, 95.2)
- moved MX33 292.4 mm to (238.1, 47.6)
- moved D29 283.1 mm to (226.0, 47.5), turned to 180 degrees
- moved MX44 270.9 mm to (276.2, 128.6)
- moved D40 269.5 mm to (264.0, 109.0), turned to 180 degrees
- moved MX41 269.2 mm to (276.2, 71.4)
- moved D38 267.8 mm to (264.0, 71.0), turned to 180 degrees
- moved MX38 266.8 mm to (257.2, 76.2)
- moved MX36 266.3 mm to (238.1, 104.8)
- moved MX29 256.5 mm to (219.1, 52.4)
- moved D39 255.9 mm to (264.0, 90.0), turned to 180 degrees
- moved MX43 250.1 mm to (276.2, 109.5)
- moved D13 245.3 mm to (102.0, 47.5), turned to 180 degrees
- moved MX23 243.3 mm to (181.0, 95.2)
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Connections:
- net ROW2 renamed COL5

Commit message: Fixed Schematic
Parts:
- D25: moved to B.Cu
- moved D25 94.7 mm to (172.8, 109.3), turned to 180 degrees
- moved MX36 21.5 mm to (227.7, 85.9)
- moved MX44 21.5 mm to (265.8, 109.7)
- moved D26 21.5 mm to (196.6, 33.1)
- moved D27 21.5 mm to (196.6, 52.1)
- moved D29 21.5 mm to (215.6, 28.6)
- moved D30 21.5 mm to (215.6, 47.6)
- moved D33 21.5 mm to (234.6, 23.6)
- moved D34 21.5 mm to (234.6, 42.6)
- moved D35 21.5 mm to (234.6, 61.6)
- moved D37 21.5 mm to (253.6, 33.1)
- moved D38 21.5 mm to (253.6, 52.1)
- moved D41 21.5 mm to (272.6, 47.6)
- moved MX12 21.5 mm to (65.8, 85.9)
- moved MX26 21.5 mm to (189.6, 38.3)
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Connections:
- D11 pad 1: COL5 -> ROW2
- D12 pad 1: COL5 -> ROW3
- D15 pad 1: COL5 -> ROW2
- D16 pad 1: COL5 -> ROW3
- D19 pad 1: COL5 -> ROW2
- D20 pad 1: COL5 -> ROW2
- D21 pad 1: COL5 -> ROW3
- D23 pad 1: COL5 -> ROW2
- D24 pad 1: COL5 -> ROW3
- D28 pad 1: COL5 -> ROW2
- D3 pad 1: COL5 -> ROW2
- D31 pad 1: COL5 -> ROW2
- D32 pad 1: COL5 -> ROW3
- D35 pad 1: COL5 -> ROW2
- D36 pad 1: COL5 -> ROW3
- D39 pad 1: COL5 -> ROW2
- D4 pad 1: COL5 -> ROW3
- D40 pad 1: COL5 -> ROW3
- D43 pad 1: COL5 -> ROW2
- D44 pad 1: COL5 -> ROW3
- D7 pad 1: COL5 -> ROW2
- D8 pad 1: COL5 -> ROW3

Commit message: Cheeky matrix optimization
Connections:
- D22 pad 1: ROW4 -> ROW1
- D25 pad 1: ROW4 -> ROW1

Commit message: Fixed Matrix
Connections:
- D20 pad 1: ROW2 -> ROW1
- D21 pad 1: ROW3 -> ROW2
- D22 pad 1: ROW1 -> ROW3
- D23 pad 1: ROW2 -> ROW1
- D24 pad 1: ROW3 -> ROW2
- D25 pad 1: ROW1 -> ROW3

Commit message: mcu traces
Parts:
- C1, C2, C3, C4, C5, C6, C7, F1, J1, R1, R2, R3, R4, R5, R6, R7, SW1, U1, U2, Y1: moved to B.Cu
- moved SW1 255.1 mm to (158.0, 66.7)
- moved C5 242.8 mm to (157.4, 87.5)
- moved C4 237.6 mm to (144.6, 82.8), turned to 180 degrees
- moved R6 173.0 mm to (155.5, 76.0)
- moved H8 169.1 mm to (158.0, 166.0)
- moved H3 169.1 mm to (137.8, 167.3)
- moved H1 169.1 mm to (114.0, 167.3)
- moved H2 169.1 mm to (125.9, 167.3)
- moved H5 169.1 mm to (131.8, 167.3)
- moved H6 169.1 mm to (120.0, 167.3)
- moved H7 169.1 mm to (108.0, 167.3)
- moved F1 164.7 mm to (156.0, 54.0), turned to -90 degrees
- moved R3 155.3 mm to (157.0, 45.8), turned to -90 degrees
- moved R1 149.3 mm to (155.5, 40.5)
- moved C2 149.3 mm to (151.8, 95.8)
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Connections:
- U2 pad 3: Net-(R5-Pad2) -> Net-(R4-Pad2)
- U2 pad 4: Net-(R4-Pad2) -> Net-(R5-Pad2)
Routing:
- net +5V: track 0.00 -> 60.2 mm, vias 0 -> 5
- net GND: track 0.00 -> 56.1 mm, vias 0 -> 2
- net DI-: track 0.00 -> 23.5 mm
- net DI+: track 0.00 -> 23.4 mm
- net Net-(J1-PadS1): track 0.00 -> 19.0 mm
- net unconnected-(U2-Pad12): track 0.00 -> 13.9 mm
- net unconnected-(U2-Pad10): track 0.00 -> 13.0 mm
- net unconnected-(U2-Pad11): track 0.00 -> 13.0 mm
- net unconnected-(U2-Pad8): track 0.00 -> 12.9 mm
- net unconnected-(U2-Pad9): track 0.00 -> 12.6 mm
- net Net-(R6-Pad1): track 0.00 -> 12.1 mm
- net Net-(R4-Pad2): track 0.00 -> 11.0 mm
- net Net-(R5-Pad2): track 0.00 -> 11.0 mm
- net D-: track 0.00 -> 10.8 mm
- net D+: track 0.00 -> 10.8 mm
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
Commit message: finished mcu routes
Parts:
- added Brd1: SSD1306, SSD1306:128x64OLED, F.Cu at (81.0, 138.1)
- moved R3 6.98 mm to (150.0, 46.1)
- moved F1 5.70 mm to (151.5, 50.5)
- moved SW1 0.33 mm to (157.7, 66.6)
Connections:
- U2 pad 18: unconnected-(U2-Pad18) -> SCL
- U2 pad 19: unconnected-(U2-Pad19) -> SDA
Routing:
- net +5V: track 60.2 -> 97.8 mm, vias 5 -> 7
- net Net-(F1-Pad1): track 0.00 -> 15.1 mm
- net Net-(R6-Pad1): track 12.1 -> 19.7 mm
- net GND: track 56.1 -> 60.1 mm, vias 2 -> 4
- net Net-(J1-PadB5): track 0.00 -> 3.92 mm
- net unconnected-(U2-Pad18): track 3.63 -> 0.00 mm
- net SCL: track 0.00 -> 3.63 mm
- net unconnected-(U2-Pad19): track 2.91 -> 0.00 mm
- net SDA: track 0.00 -> 2.91 mm
- added copper zone on B.Cu, net GND
- added copper zone on F.Cu, net GND

Commit message: Wired Matrix
Routing:
- net ROW3: track 0.00 -> 252.3 mm
- net ROW1: track 0.00 -> 248.3 mm
- net ROW2: track 0.00 -> 238.8 mm
- net ROW0: track 0.00 -> 186.7 mm
- net COL9: track 0.00 -> 57.2 mm
- net COL2: track 0.00 -> 57.2 mm
- net COL11: track 0.00 -> 57.2 mm
- net COL0: track 0.00 -> 57.2 mm
- net COL10: track 0.00 -> 57.1 mm
- net COL1: track 0.00 -> 57.1 mm
- net COL8: track 0.00 -> 57.1 mm
- net COL3: track 0.00 -> 57.1 mm
- net COL6: track 0.00 -> 49.0 mm
- net COL5: track 0.00 -> 48.0 mm
- net COL7: track 0.00 -> 38.1 mm
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
Commit message: Added 2 1u options for space
Parts:
- added D45: D_Small, Diode_SMD:D_SOD-123, B.Cu at (111.9, 92.9)
- added D46: D_Small, Diode_SMD:D_SOD-123, B.Cu at (131.0, 92.9)
- added D47: D_Small, Diode_SMD:D_SOD-123, B.Cu at (178.6, 92.9)
- added D48: D_Small, Diode_SMD:D_SOD-123, B.Cu at (198.4, 92.9)
- added MX45: MX-NoLED, MX_Only:MXOnly-1U-NoLED, F.Cu at (104.8, 100.0)
- added MX46: MX-NoLED, MX_Only:MXOnly-1U-NoLED, F.Cu at (123.8, 100.0)
- added MX47: MX-NoLED, MX_Only:MXOnly-1U-NoLED, F.Cu at (171.4, 100.0)
- added MX48: MX-NoLED, MX_Only:MXOnly-1U-NoLED, F.Cu at (190.5, 100.0)
- moved Brd1 12.8 mm to (76.2, 150.0)
- moved D21 2.34 mm to (121.0, 92.9)
- moved D24 2.34 mm to (188.0, 92.9)
Connections:
- D20 pad 1: ROW1 -> ROW0
- D21 pad 1: ROW2 -> ROW1
- D22 pad 1: ROW3 -> ROW2
- D23 pad 1: ROW1 -> ROW0
- D24 pad 1: ROW2 -> ROW1
- D25 pad 1: ROW3 -> ROW2
Routing:
- net ROW3: track 252.3 -> 145.0 mm
- net ROW1: track 248.3 -> 186.6 mm
- net COL5: track 48.0 -> 0.00 mm
- net ROW2: track 238.8 -> 192.4 mm
- net COL6: track 49.0 -> 9.51 mm
- net Net-(D21-Pad2): track 2.60 -> 0.00 mm
- net Net-(D24-Pad2): track 2.93 -> 0.40 mm
