File: Hydra/Hydra.kicad_pcb (KiCad board)
At the start: 2 copper layers, 125 parts, among them J1 USB_C_Receptacle_USB2.0, SW1 SW_Push, U1 USBLC6-2SC6, U2 ATmega32U4-M, Y1 16MHz

Commit message: stuff lol
Parts:
- moved Brd1 93.0 mm to (147.6, 90.5), turned to 180 degrees
Changed lines of the file:
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@@
   )
   (footprint "SSD1306:128x64OLED" (layer "F.Cu")
-    (at 76.2 150.01875)
+    (at 147.6375 90.4875 180)
     (property "Sheetfile" "Hydra.kicad_sch")
     (property "Sheetname" "")
@@
     (fp_line (start -12.978 7.595) (end -12.978 -9.005) (layer "F.SilkS") (width 0.12))
     (fp_line (start -13.4 -12.3) (end 14 -12.3) (layer "F.SilkS") (width 0.12))
-    (pad "1" thru_hole oval locked (at -3.62 -10.6 90) (size 2 1.6) (drill 1) (layers *.Cu *.Mask)
+    (pad "1" thru_hole oval locked (at -3.62 -10.6 270) (size 2 1.6) (drill 1) (layers *.Cu *.Mask)
       (net 2 "GND") (pinfunction "GND") (pintype "input"))
-    (pad "2" thru_hole oval locked (at -1.08 -10.6 90) (size 2 1.6) (drill 1) (layers *.Cu *.Mask)
+    (pad "2" thru_hole oval locked (at -1.08 -10.6 270) (size 2 1.6) (drill 1) (layers *.Cu *.Mask)
       (net 1 "+5V") (pinfunction "VCC") (pintype "input"))
-    (pad "3" thru_hole oval locked (at 1.46 -10.6 90) (size 2 1.6) (drill 1) (layers *.Cu *.Mask)
+    (pad "3" thru_hole oval locked (at 1.46 -10.6 270) (size 2 1.6) (drill 1) (layers *.Cu *.Mask)
       (net 91 "SCL") (pinfunction "SCL") (pintype "input"))
-    (pad "4" thru_hole oval locked (at 4 -10.6 90) (size 2 1.6) (drill 1) (layers *.Cu *.Mask)
+    (pad "4" thru_hole oval locked (at 4 -10.6 270) (size 2 1.6) (drill 1) (layers *.Cu *.Mask)
       (net 90 "SDA") (pinfunction "SDA") (pintype "input"))
   )
