File: Hydra/Hydra.kicad_pcb (KiCad board)
At the start: 2 copper layers, 125 parts, among them J1 USB_C_Receptacle_USB2.0, SW1 SW_Push, U1 USBLC6-2SC6, U2 ATmega32U4-M, Y1 16MHz

Commit message: routed switch matrix and oled
Parts:
- moved D48 19.7 mm to (188.0, 109.6), turned to 90 degrees
- moved D46 19.4 mm to (121.2, 109.6), turned to 90 degrees
- moved D24 18.7 mm to (173.8, 105.0), turned to 0 degrees
- moved D21 7.97 mm to (113.4, 90.4)
- moved D22 6.44 mm to (131.2, 108.9), turned to -90 degrees
- moved D1 6.44 mm to (31.2, 47.4), turned to -90 degrees
- moved D2 6.44 mm to (31.2, 66.4), turned to -90 degrees
- moved D3 6.44 mm to (31.2, 85.4), turned to -90 degrees
- moved D4 6.44 mm to (31.2, 104.4), turned to -90 degrees
- moved D11 6.44 mm to (69.2, 61.4), turned to -90 degrees
- moved D5 6.44 mm to (50.2, 32.9), turned to -90 degrees
- moved D6 6.44 mm to (50.2, 51.9), turned to -90 degrees
- moved D7 6.44 mm to (50.2, 71.4), turned to -90 degrees
- moved D8 6.44 mm to (50.2, 90.4), turned to -90 degrees
- moved D10 6.44 mm to (69.2, 42.4), turned to -90 degrees
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Routing:
- net ROW0: track 186.7 -> 375.6 mm
- net ROW3: track 145.0 -> 320.6 mm
- net ROW1: track 186.6 -> 359.2 mm
- net ROW2: track 192.4 -> 324.6 mm
- net COL5: track 0.00 -> 53.6 mm
- net COL6: track 9.51 -> 61.3 mm
- net COL7: track 38.1 -> 65.4 mm
- net SDA: track 2.91 -> 23.0 mm
- net COL4: track 38.1 -> 57.9 mm
- net SCL: track 3.63 -> 21.8 mm
- net Net-(D21-Pad2): track 0.00 -> 14.8 mm
- net +5V: track 97.8 -> 108.6 mm, vias 7 -> 8
- net Net-(D47-Pad2): track 0.00 -> 5.04 mm
- net Net-(D46-Pad2): track 0.00 -> 3.06 mm
- net Net-(D23-Pad2): track 2.91 -> 0.00 mm
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